Commit message: changed wheel meshs to gazebo def
add better performance

File: catvehicle.xacro (robot description, xacro)
@@ -71,4 +71,5 @@
     <!-- Inertial tensor of car body has been taken from meshlab after
     analyzing the 3D structure of car body -->
+    <!-- old inertias
     <xacro:property name="base_mass_ixx" value="347.195805"/>
     <xacro:property name="base_mass_ixy" value="-11.4914985"/>
@@ -77,4 +78,12 @@
     <xacro:property name="base_mass_iyz" value="3.97814264"/>
     <xacro:property name="base_mass_izz" value="2529.41827"/>
+    -->
+<!-- estimated sprung inertia of the 2019 racing vehicle-->
+    <xacro:property name="base_mass_ixx" value="19.118"/>
+    <xacro:property name="base_mass_ixy" value="-1.36778"/>
+    <xacro:property name="base_mass_ixz" value="-10.4111"/>
+    <xacro:property name="base_mass_iyy" value="111.9943"/>
+    <xacro:property name="base_mass_iyz" value="0.1475"/>
+    <xacro:property name="base_mass_izz" value="108.489"/>
     <!--changed all of these, here are the originals
      <xacro:property name="tyre_x" value="1.05"/>
@@ -204,8 +213,9 @@
     <link name="back_right_wheel_link">
         <collision>
-            <origin xyz="0 0 0" rpy="0 0 -${PI}"/>
-            <geometry>
-                <!--<cylinder length="${tyre_length}" radius="${tyre_radius}"/-->
-                <mesh filename="package://catvehicle/meshes/EE88_wheel2.dae"/>
+            <!--origin xyz="0 0 0" rpy="0 0 -${PI}"/-->
+	    <origin xyz="0 0 0" rpy="${PI/2} 0 0"/>
+            <geometry>
+                <cylinder length="${tyre_length}" radius="${tyre_radius}"/>
+                <!--mesh filename="package://catvehicle/meshes/EE88_wheel2.dae"/-->
             </geometry>
             <surface>
@@ -259,8 +269,9 @@
     <link name="back_left_wheel_link">
         <collision>
-            <origin xyz="0 0 0" rpy="0 0 0"/>
-            <geometry>
-                <!--cylinder length="${tyre_length}" radius="${tyre_radius}"/-->
-                <mesh filename="package://catvehicle/meshes/EE88_wheel2.dae"/>
+            <!--origin xyz="0 0 0" rpy="0 0 0"/-->
+	    <origin xyz="0 0 0" rpy="${PI/2} 0 0"/>
+            <geometry>
+                <cylinder length="${tyre_length}" radius="${tyre_radius}"/>
+                <!--mesh filename="package://catvehicle/meshes/EE88_wheel2.dae"/-->
             </geometry>
             <surface>
@@ -343,9 +354,9 @@
     <link name="front_right_wheel_link">
         <collision>
-            <!--origin xyz="0 0 0" rpy="${PI/2} 0 0"/-->
-            <origin xyz="0 0.10 0" rpy="0 0 ${-PI}"/>
-            <geometry>
-                <!--cylinder length="${tyre_length}" radius="${tyre_radius}"/-->
-                <mesh filename="package://catvehicle/meshes/EE88_wheel2.dae"/>
+            <origin xyz="0 0 0" rpy="${PI/2} 0 0"/>
+            <!--origin xyz="0 0.10 0" rpy="0 0 ${-PI}"/-->
+            <geometry>
+                <cylinder length="${tyre_length}" radius="${tyre_radius}"/>
+                <!--mesh filename="package://catvehicle/meshes/EE88_wheel2.dae"/-->
             </geometry>
             <surface>
@@ -431,9 +442,9 @@
         <parent link="front_left_wheel_joint"/>
         <collision>
-            <!--origin xyz="0 0 0" rpy="${PI/2} 0 0"/-->
-            <origin xyz="0 -0.10 0" rpy="0 0 0"/>
-            <geometry>
-                <!--cylinder length="${tyre_length}" radius="${tyre_radius}"/-->
-                <mesh filename="package://catvehicle/meshes/EE88_wheel2.dae"/>
+            <origin xyz="0 0 0" rpy="${PI/2} 0 0"/>
+            <!--origin xyz="0 -0.10 0" rpy="0 0 0"/-->
+            <geometry>
+                <cylinder length="${tyre_length}" radius="${tyre_radius}"/>
+                <!--<mesh filename="package://catvehicle/meshes/EE88_wheel2.dae"/>-->
             </geometry>
             <surface>
