Commit message: fix for model and camera frame

File: urdf/catvehicle.xacro (robot description, xacro)
@@ -29,6 +29,6 @@
 -->
 <robot name="$(arg roboname)" xmlns:xacro="http://www.ros.org/wiki/xacro">
-    <xacro:arg name="camera_left" default="true"/>
-    <xacro:arg name="camera_right" default="true"/>
+    <xacro:arg name="camera_left" default="false"/>
+    <xacro:arg name="camera_right" default="false"/>
     <xacro:arg name="triclops" default="true"/>
     <xacro:arg name="velodyne_points" default="true"/>
@@ -58,14 +58,15 @@
     <!-- Edited to length given by design spec sheet, was 4.4324092962 -->
     <xacro:property name="car_to_bumper" value="2.900"/>
-    <xacro:property name="car_COM_x" value="1.00"/>
+    <xacro:property name="car_COM_x" value="1.50"/>
     <xacro:property name="car_COM_y" value="0.000"/>
     <xacro:property name="car_COM_z" value="0.260"/>
     <!-- We are assuming that front bumper's height is half of the car's
     bounding box height -->
-    <xacro:property name="front_bumper_height" value="${car_height/2}"/>
+    <xacro:property name="front_bumper_height" value="0.3"/>
     <!--This is the car tread, i.e distance between right and left front wheels-->
     <!-- Edited to width given by design spec sheet, was 1.290-->
     <xacro:property name="car_width" value="1.140"/>
-    <xacro:property name="car_width_offset" value="0.05"/>
+    <xacro:property name="car_width_offset" value="0.10"/>
+    <xacro:property name="car_tyre_offset" value="0.1905"/>
     <!-- Inertial tensor of car body has been taken from meshlab after
     analyzing the 3D structure of car body -->
@@ -83,8 +84,8 @@
     <xacro:property name="tyre_r" value="0.66"/>-->
     <xacro:property name="tyre_x" value="1.05"/>
-    <xacro:property name="tyre_front_x" value="1.55"/>
-    <xacro:property name="tyre_back_x" value="0"/>
-    <xacro:property name="tyre_y" value="0.590"/>
-    <xacro:property name="tyre_r" value="0.10"/>
+    <xacro:property name="tyre_front_x" value="1.9500"/>
+    <xacro:property name="tyre_back_x" value="0.45"/>
+    <xacro:property name="tyre_y" value="0.420"/> <!--edited to 1.590 from 0.590-->
+    <xacro:property name="tyre_r" value="0.15"/>
     <!--Below is the thickness of the car's tyre-->
     <!-- edited for eletric vehicles 18inch/7.5 inch wheels-->
@@ -164,5 +165,5 @@
             <origin xyz="0 0 ${base_height}" rpy="0 0 0"/>
             <geometry>
-                <mesh filename="package://catvehicle/meshes/EE88_1.dae"/>
+                <mesh filename="package://catvehicle/meshes/EE88_2.dae"/>
             </geometry>
         </collision>
@@ -171,5 +172,5 @@
             <geometry>
 		<!-- edited "package://catvehicle/meshes/ford_escape_no_wheels_2.dae"/> to below-->
-                <mesh filename="package://catvehicle/meshes/EE88_1.dae"/>
+                <mesh filename="package://catvehicle/meshes/EE88_2.dae"/>
             </geometry>
         </visual>
@@ -203,8 +204,8 @@
     <link name="back_right_wheel_link">
         <collision>
-            <origin xyz="0 0 0" rpy="0 0 ${PI/2}"/>
+            <origin xyz="0 0 0" rpy="0 0 -${PI}"/>
             <geometry>
                 <!--<cylinder length="${tyre_length}" radius="${tyre_radius}"/-->
-                <mesh filename="package://catvehicle/meshes/EE88_wheel1.dae"/>
+                <mesh filename="package://catvehicle/meshes/EE88_wheel2.dae"/>
             </geometry>
             <surface>
@@ -229,10 +230,10 @@
         </collision>
         <visual>
-            <origin xyz="0 0 0" rpy="0 0 ${PI/2}"/>
+            <origin xyz="0 0 0" rpy="0 0 -${PI}"/>
             <!--origin xyz="0 ${car_width_offset*2} 0.0" rpy="0 0 ${-PI/2}"/-->
             <geometry>
                 <!--cylinder length="${tyre_length}" radius="${tyre_radius}"/>
                 <scale xyz="1 1 1"/-->
-                <mesh scale="1 1 1" filename="package://catvehicle/meshes/EE88_wheel1.dae"/>
+                <mesh scale="1 1 1" filename="package://catvehicle/meshes/EE88_wheel2.dae"/>
             </geometry>
         </visual>
@@ -258,8 +259,8 @@
     <link name="back_left_wheel_link">
         <collision>
-            <origin xyz="0 0 0" rpy="0 0 ${PI/2}"/>
+            <origin xyz="0 0 0" rpy="0 0 0"/>
             <geometry>
                 <!--cylinder length="${tyre_length}" radius="${tyre_radius}"/-->
-                <mesh filename="package://catvehicle/meshes/EE88_wheel1.dae"/>
+                <mesh filename="package://catvehicle/meshes/EE88_wheel2.dae"/>
             </geometry>
             <surface>
@@ -284,9 +285,9 @@
         </collision>
         <visual>
-            <origin xyz="0 0 0" rpy="0 0 ${PI/2}"/>
+            <origin xyz="0 0 0" rpy="0 0 0"/>
             <!--origin xyz="0 ${-car_width_offset*2} 0.0" rpy="0 0 ${PI/2}"/-->
             <geometry>
                 <!--cylinder length="${tyre_length}" radius="${tyre_radius}"/-->
-                <mesh scale="1 1 1" filename="package://catvehicle/meshes/EE88_wheel1.dae"/>
+                <mesh scale="1 1 1" filename="package://catvehicle/meshes/EE88_wheel2.dae"/>
             </geometry>
         </visual>
@@ -304,5 +305,5 @@
         <parent link="base_link"/>
         <child link="front_right_steering_link"/>
-        <origin xyz="${tyre_front_x} ${-car_width/2 - 2*str_length} ${tyre_r}" rpy="0 0 0"/>
+        <origin xyz="${tyre_front_x} ${-tyre_y-car_width_offset} ${tyre_r}" rpy="0 0 0"/>
         <axis xyz="0 0 1"/>
         <limit effort="10000" lower="${-str_angle}" upper="${str_angle}" velocity="1000"/>
@@ -343,8 +344,8 @@
         <collision>
             <!--origin xyz="0 0 0" rpy="${PI/2} 0 0"/-->
-            <origin xyz="0 0 0" rpy="0 0 ${-PI/2}"/>
+            <origin xyz="0 0.10 0" rpy="0 0 ${-PI}"/>
             <geometry>
                 <!--cylinder length="${tyre_length}" radius="${tyre_radius}"/-->
-                <mesh filename="package://catvehicle/meshes/EE88_wheel1.dae"/>
+                <mesh filename="package://catvehicle/meshes/EE88_wheel2.dae"/>
             </geometry>
             <surface>
@@ -370,9 +371,9 @@
         <visual>
             <!--origin xyz="0 0 0" rpy="${PI/2} 0 0"/-->
-            <origin xyz="0 ${car_width_offset*2} 0.0" rpy="0 0 ${PI/2}"/>
+            <origin xyz="0 0.10 0" rpy="0 0 ${-PI}"/>
             <geometry>
                 <!--cylinder length="${tyre_length}" radius="${tyre_radius}"/>
                 <scale xyz="1 1 1"/-->
-                <mesh scale="1 1 1" filename="package://catvehicle/meshes/EE88_wheel1.dae"/>
+                <mesh scale="1 1 1" filename="package://catvehicle/meshes/EE88_wheel2.dae"/>
                 </geometry>
         </visual>
@@ -390,5 +391,5 @@
         <parent link="base_link"/>
         <child link="front_left_steering_link"/>
-        <origin xyz="${tyre_front_x} ${car_width/2 + 2*str_length} ${tyre_r}" rpy="0 0 0"/>
+        <origin xyz="${tyre_front_x} ${tyre_y+car_width_offset} ${tyre_r}" rpy="0 0 0"/>
         <axis xyz="0 0 1"/>
         <limit effort="10000" lower="${-str_angle}" upper="${str_angle}" velocity="1000"/>
@@ -431,8 +432,8 @@
         <collision>
             <!--origin xyz="0 0 0" rpy="${PI/2} 0 0"/-->
-            <origin xyz="0 0 0" rpy="0 0 ${-PI/2}"/>
+            <origin xyz="0 -0.10 0" rpy="0 0 0"/>
             <geometry>
                 <!--cylinder length="${tyre_length}" radius="${tyre_radius}"/-->
-                <mesh filename="package://catvehicle/meshes/EE88_wheel1.dae"/>
+                <mesh filename="package://catvehicle/meshes/EE88_wheel2.dae"/>
             </geometry>
             <surface>
@@ -458,8 +459,8 @@
         <visual>
             <!--origin xyz="0 0 0" rpy="${PI/2} 0 0"/-->
-            <origin xyz="0 ${-car_width_offset*2} 0.0" rpy="0 0 ${-PI/2}"/>
+            <origin xyz="0 -0.10 0.0" rpy="0 0 0"/>
             <geometry>
             <!--cylinder length="${tyre_length}" radius="${tyre_radius}"/-->
-            <mesh scale="1 1 1" filename="package://catvehicle/meshes/EE88_wheel1.dae"/>
+            <mesh scale="1 1 1" filename="package://catvehicle/meshes/EE88_wheel2.dae"/>
             </geometry>
         </visual>
@@ -475,5 +476,5 @@
     <!-- front laser-->
     <joint name="front_laser_joint" type="fixed">
-        <origin xyz="${car_to_bumper/2 + front_laser_size} 0 ${front_bumper_height + front_laser_size/2 + 0.90}" rpy="0 0 0"/>
+        <origin xyz="${car_to_bumper + 0.1} 0 ${front_bumper_height + 0.15}" rpy="0 0 0"/>
         <axis xyz="0 0 1"/>
         <parent link="base_link"/>
@@ -485,5 +486,5 @@
                 <origin xyz="0 0 0" rpy="0 0.0 0"/>
                 <geometry>
-                    <box size="${front_laser_size} ${front_laser_size} ${front_laser_size}"/>
+                    <box size="0.01 0.01 0.01"/>
                 </geometry>
             </collision>
@@ -502,4 +503,5 @@
             </inertial>
             </link>
+<!--
     <joint name="camera_right_joint" type="fixed">
     <origin xyz="-0.75 -${car_width/2} ${0.725 + camera_box/2 + 1.25}" rpy="0 0 -${PI/2}"/>
@@ -552,10 +554,21 @@
         </inertial>
     </link>
+-->
     <joint name="triclops" type="fixed">
-    <origin xyz="0.75 0 ${0.725 + sensor_box/2 + 1.2}" rpy="0 0 0"/>
+    <origin xyz="0.98 0 1.02" rpy="0 0 0"/> <!-- edited origin to line up with vehicle -->
         <axis xyz="0 0 1"/>
         <parent link="base_link"/>
         <child link="triclops_link"/>
     </joint>
+	<joint name="triclops_optical_joint" type="fixed">
+    <!-- these values have to be these values otherwise the gazebo camera
+        image won't be aligned properly with the frame it is supposedly
+        originating from -->
+    <origin xyz="0 0 0" rpy="${-pi/2} 0 ${-pi/2}"/>
+    	<parent link="triclops_link"/>
+    	<child link="triclops_link_optical"/>
+  	</joint>
+    <link name="triclops_link_optical">
+    </link>
     <link name="triclops_link">
         <collision>
@@ -578,7 +591,7 @@
     </link>
         <joint name="velodyne_joint" type="fixed">
-            <origin xyz="-0.5 0 ${sensor_box/2 + 0.01}" rpy="0 0 0"/>
+            <origin xyz="${car_to_bumper + 0.05} 0 ${front_bumper_height + 0.1}" rpy="0 0 0"/>
             <axis xyz="0 0 1"/>
-            <parent link="triclops_link"/>
+            <parent link="base_link"/>
             <child link="velodyne_link"/>
         </joint>

Commit message: Inertia changes makes car much more driveable

File: urdf/catvehicle.xacro (robot description, xacro)
@@ -71,4 +71,5 @@
     <!-- Inertial tensor of car body has been taken from meshlab after
     analyzing the 3D structure of car body -->
+    <!-- old inertias
     <xacro:property name="base_mass_ixx" value="347.195805"/>
     <xacro:property name="base_mass_ixy" value="-11.4914985"/>
@@ -77,4 +78,12 @@
     <xacro:property name="base_mass_iyz" value="3.97814264"/>
     <xacro:property name="base_mass_izz" value="2529.41827"/>
+    -->
+<!-- estimated sprung inertia of the 2019 racing vehicle-->
+    <xacro:property name="base_mass_ixx" value="19.118"/>
+    <xacro:property name="base_mass_ixy" value="-1.36778"/>
+    <xacro:property name="base_mass_ixz" value="-10.4111"/>
+    <xacro:property name="base_mass_iyy" value="111.9943"/>
+    <xacro:property name="base_mass_iyz" value="0.1475"/>
+    <xacro:property name="base_mass_izz" value="108.489"/>
     <!--changed all of these, here are the originals
      <xacro:property name="tyre_x" value="1.05"/>

Commit message: improved wheel dynamics

File: urdf/catvehicle.xacro (robot description, xacro)
@@ -213,8 +213,9 @@
     <link name="back_right_wheel_link">
         <collision>
-            <origin xyz="0 0 0" rpy="0 0 -${PI}"/>
-            <geometry>
-                <!--<cylinder length="${tyre_length}" radius="${tyre_radius}"/-->
-                <mesh filename="package://catvehicle/meshes/EE88_wheel2.dae"/>
+            <!--origin xyz="0 0 0" rpy="0 0 -${PI}"/-->
+	    <origin xyz="0 0 0" rpy="${PI/2} 0 0"/>
+            <geometry>
+                <cylinder length="${tyre_length}" radius="${tyre_radius}"/>
+                <!--mesh filename="package://catvehicle/meshes/EE88_wheel2.dae"/-->
             </geometry>
             <surface>
@@ -268,8 +269,9 @@
     <link name="back_left_wheel_link">
         <collision>
-            <origin xyz="0 0 0" rpy="0 0 0"/>
-            <geometry>
-                <!--cylinder length="${tyre_length}" radius="${tyre_radius}"/-->
-                <mesh filename="package://catvehicle/meshes/EE88_wheel2.dae"/>
+            <!--origin xyz="0 0 0" rpy="0 0 0"/-->
+	    <origin xyz="0 0 0" rpy="${PI/2} 0 0"/>
+            <geometry>
+                <cylinder length="${tyre_length}" radius="${tyre_radius}"/>
+                <!--mesh filename="package://catvehicle/meshes/EE88_wheel2.dae"/-->
             </geometry>
             <surface>
@@ -352,9 +354,9 @@
     <link name="front_right_wheel_link">
         <collision>
-            <!--origin xyz="0 0 0" rpy="${PI/2} 0 0"/-->
-            <origin xyz="0 0.10 0" rpy="0 0 ${-PI}"/>
-            <geometry>
-                <!--cylinder length="${tyre_length}" radius="${tyre_radius}"/-->
-                <mesh filename="package://catvehicle/meshes/EE88_wheel2.dae"/>
+            <origin xyz="0 0 0" rpy="${PI/2} 0 0"/>
+            <!--origin xyz="0 0.10 0" rpy="0 0 ${-PI}"/-->
+            <geometry>
+                <cylinder length="${tyre_length}" radius="${tyre_radius}"/>
+                <!--mesh filename="package://catvehicle/meshes/EE88_wheel2.dae"/-->
             </geometry>
             <surface>
@@ -440,9 +442,9 @@
         <parent link="front_left_wheel_joint"/>
         <collision>
-            <!--origin xyz="0 0 0" rpy="${PI/2} 0 0"/-->
-            <origin xyz="0 -0.10 0" rpy="0 0 0"/>
-            <geometry>
-                <!--cylinder length="${tyre_length}" radius="${tyre_radius}"/-->
-                <mesh filename="package://catvehicle/meshes/EE88_wheel2.dae"/>
+            <origin xyz="0 0 0" rpy="${PI/2} 0 0"/>
+            <!--origin xyz="0 -0.10 0" rpy="0 0 0"/-->
+            <geometry>
+                <cylinder length="${tyre_length}" radius="${tyre_radius}"/>
+                <!--<mesh filename="package://catvehicle/meshes/EE88_wheel2.dae"/>-->
             </geometry>
             <surface>

Commit message: atempting to get loop closure acurate
also fixed imu link and transform i

File: urdf/catvehicle.xacro (robot description, xacro)
@@ -175,4 +175,5 @@
             <geometry>
                 <mesh filename="package://catvehicle/meshes/EE88_2.dae"/>
+            <!--<box size="${camera_box} ${camera_box} ${camera_box}"/>  very small box collision for the vehicle to improve gazebo sim times-->
             </geometry>
         </collision>

Commit message: Updated car model with gps
also disabled obstacle stopper

File: urdf/catvehicle.xacro (robot description, xacro)
@@ -35,4 +35,5 @@
     <xacro:arg name="laser_points" default="true"/>
     <xacro:arg name="imu" default="true"/>
+    <xacro:arg name="gps" default="true"/>
     <xacro:property name="velodyne_points" value="$(arg velodyne_points)"/>
     <xacro:property name="laser_points" value="$(arg laser_points)"/>
@@ -41,4 +42,5 @@
     <xacro:property name="triclops" value="$(arg triclops)"/>
     <xacro:property name="imu" value="$(arg imu)"/>
+    <xacro:property name="gps" value="$(arg gps)"/>
     <xacro:property name="camera_box" value="0.1"/>
     <xacro:property name="sensor_box" value="0.25"/>
@@ -169,4 +171,7 @@
         <xacro:include filename="$(find catvehicle)/urdf/catvehicle_imu.gazebo"/>
     </xacro:if>
+    <xacro:if value="${gps}">
+        <xacro:include filename="$(find catvehicle)/urdf/catvehicle_gps.gazebo"/>
+    </xacro:if>
     <!--Car Body-->
     <link name="base_link">
@@ -189,10 +194,10 @@
         <parent link="base_link"/>
         <child link="main_mass"/>
-        <origin xyz="0 0 0" rpy="0 0 0"/>
+        <origin xyz="${car_COM_x} ${car_COM_y} ${car_COM_z}" rpy="0 0 0"/>
     </joint>
     <link name="main_mass" type="fixed">
         <parent link="inertial_joint"/>
         <inertial>
-            <origin xyz="${car_COM_x} ${car_COM_y} ${car_COM_z}" rpy="0 0 0"/> <!-- This is the center of mass of Car Body-->
+            <origin xyz="0 0 0" rpy="0 0 0"/> <!-- This is the center of mass of Car Body-->
             <mass value="${base_mass}"/>
             <inertia
@@ -488,5 +493,5 @@
     <!-- front laser-->
     <joint name="front_laser_joint" type="fixed">
-        <origin xyz="${car_to_bumper + 0.1} 0 ${front_bumper_height + 0.15}" rpy="0 0 0"/>
+        <origin xyz="${car_to_bumper + 0.1} 0 ${front_bumper_height - 0.25}" rpy="0 0 0"/>
         <axis xyz="0 0 1"/>
         <parent link="base_link"/>
@@ -603,5 +608,5 @@
     </link>
         <joint name="velodyne_joint" type="fixed">
-            <origin xyz="${car_to_bumper + 0.05} 0 ${front_bumper_height + 0.1}" rpy="0 0 0"/>
+            <origin xyz="${car_to_bumper + 0.05} 0 ${front_bumper_height - 0.1}" rpy="0 0 0"/>
             <axis xyz="0 0 1"/>
             <parent link="base_link"/>

Commit message: added velodyne lidar

File: urdf/catvehicle.xacro (robot description, xacro)
@@ -608,6 +608,6 @@
     </link>
         <joint name="velodyne_joint" type="fixed">
-            <origin xyz="${car_to_bumper + 0.05} 0 ${front_bumper_height - 0.1}" rpy="0 0 0"/>
-            <axis xyz="0 0 1"/>
+            <origin xyz="${car_to_bumper + 0.05} 0 ${front_bumper_height - 0.1}" rpy="0 0.008726 0"/> tilted down 5 degrees
+            <axis xyz="0 0 0"/>
             <parent link="base_link"/>
             <child link="velodyne_link"/>
